File: V-00756-00.brd (EAGLE design)
At the start: 43 x 70 mm, 19 parts, among them IC1 MEGA8-AI, IC2 MAX481CSA, Q1 14.7456MHz

Commit message: v.2.0
Parts:
- added C7, C8: 100n, #PaJa_31:1206
- added U$2: (no value), frames:A4L-LOC
- IC2: value MAX481CSA -> MAX481
- IO1: value TL431SOT23 -> TL431
- IO2: value LF50CDT -> 78M05
- moved K2 7.07 mm to (32.0, 61.0)
- moved R3 5.00 mm to (35.2, 47.5)
- moved D1 2.97 mm to (10.6, 23.4)
- moved C3 2.40 mm to (9.10, 41.8)
- moved C4 2.40 mm to (9.10, 46.8)
- moved Q1 2.40 mm to (12.7, 44.3)
Connections:
- net +5V: now also C7.2, C8.2, U$1.2; no longer U$1.4
- net GND: now also C7.1, C8.1
- net P_MISO: now also U$1.5; no longer U$1.3
- net P_SCK: now also U$1.4; no longer U$1.2
- net RESET: now also U$1.3; no longer U$1.5
Routing:
- net INT_LOCK_0: track 34.6 -> 45.2 mm, vias 3 -> 1
- net +5V: track 64.6 -> 70.0 mm
- net RESET: track 40.6 -> 35.4 mm
- net GND: track 5.09 -> 9.89 mm, vias 1 -> 3
- net P_MISO: track 14.9 -> 18.9 mm
- net +24V: track 9.46 -> 13.1 mm
- net P_SCK: track 12.4 -> 15.9 mm
- net XTAL2: track 7.06 -> 9.46 mm
- net XTAL1: track 7.06 -> 9.46 mm
Other:
- board text added: "00"
- board text added: "DPS pro smerovac se dvema interlocky"
- board text added: "Top"
