File: V-00756-00.sch (EAGLE design)
At the start: 19 parts, among them IC1 MEGA8-AI, IC2 MAX481CSA, Q1 14.7456MHz

Commit message: v.2.0
Parts:
- added C7, C8: 100n, #PaJa_31:C-KER_1206
- IC2: value MAX481CSA -> MAX481
- IO1: value TL431SOT23 -> TL431
- IO2: value LF50CDT -> 78M05
Connections:
- net +5V: now also C7.2, C8.2
- net GND: now also C7.1, C8.1
Other:
- note added: "Smerovac, s dvema interlocky RS485 -> TTL"
- note removed: "Ovládání ofuku pres RS485 -> 5TTL"
Changed lines of the file:
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@@
 <parts>
 <part name="FRAME1" library="frames" deviceset="A4L-LOC" device=""/>
-<part name="IC2" library="maxim" deviceset="MAX481CSA" device=""/>
-<part name="IO1" library="references" deviceset="TL431" device="SOT23"/>
+<part name="IC2" library="maxim" deviceset="MAX481CSA" device="" value="MAX481"/>
+<part name="IO1" library="references" deviceset="TL431" device="SOT23" value="TL431"/>
 <part name="C1" library="#PaJa_31" deviceset="C-KER" device="_1206" value="100n"/>
 <part name="R1" library="#PaJa_31" deviceset="R" device="_1206" value="1k"/>
@@
 <part name="C4" library="#PaJa_31" deviceset="C-KER" device="_0805" value="27nF"/>
 <part name="D1" library="diode" deviceset="MBRS3*0T3" device="" technology="4"/>
-<part name="IO2" library="#PaJa_31" deviceset="LF_C" device="DT" value="LF50CDT"/>
+<part name="IO2" library="#PaJa_31" deviceset="LF_C" device="DT" value="78M05"/>
 <part name="C5" library="#PaJa_31" deviceset="C-KER" device="_1206" value="10uF"/>
 <part name="C6" library="#PaJa_31" deviceset="C-KER" device="_1206" value="100n"/>
@@
 <part name="K2" library="#PaJa_konektory" deviceset="PSH02-02" device="W"/>
 <part name="K3" library="#PaJa_konektory" deviceset="PSH02-02" device="W"/>
+<part name="C7" library="#PaJa_31" deviceset="C-KER" device="_1206" value="100n"/>
+<part name="C8" library="#PaJa_31" deviceset="C-KER" device="_1206" value="100n"/>
 </parts>
 <sheets>
 <sheet>
 <plain>
-<text x="127" y="12.7" size="2.54" layer="94">Ovládání ofuku pres
-RS485 -&gt; 5TTL</text>
+<text x="127" y="12.7" size="2.54" layer="94">Smerovac, s dvema interlocky
+RS485 -&gt; TTL</text>
 <text x="246.38" y="5.08" size="2.54" layer="94">00</text>
 </plain>
@@
 <instance part="K2" gate="KON" x="187.96" y="139.7" rot="R270"/>
 <instance part="K3" gate="KON" x="187.96" y="127" rot="R270"/>
+<instance part="C7" gate="C" x="60.96" y="30.48" rot="R90"/>
+<instance part="C8" gate="C" x="73.66" y="30.48" rot="R90"/>
 </instances>
 <busses>
@@
 <label x="78.74" y="111.76" size="1.016" layer="95" font="vector" ratio="10" rot="R180" xref="yes"/>
 <junction x="81.28" y="111.76"/>
+</segment>
+<segment>
+<pinref part="C7" gate="C" pin="2"/>
+<wire x1="60.96" y1="33.02" x2="60.96" y2="35.56" width="0.1524" layer="91"/>
+<label x="60.96" y="35.56" size="1.016" layer="95" ratio="10" rot="R180" xref="yes"/>
+</segment>
+<segment>
+<pinref part="C8" gate="C" pin="2"/>
+<wire x1="73.66" y1="33.02" x2="73.66" y2="35.56" width="0.1524" layer="91"/>
+<label x="73.66" y="35.56" size="1.016" layer="95" ratio="10" rot="R180" xref="yes"/>
 </segment>
 </net>
@@
 <label x="180.34" y="124.46" size="1.016" layer="95" ratio="10" rot="R180" xref="yes"/>
 </segment>
-</net>
+<segment>
+<pinref part="C7" gate="C" pin="1"/>
+<wire x1="60.96" y1="25.4" x2="60.96" y2="22.86" width="0.1524" layer="91"/>
+<label x="60.96" y="22.86" size="1.016" layer="95" ratio="10" rot="R180" xref="yes"/>
+</segment>
+<segment>
+<pinref part="C8" gate="C" pin="1"/>
+<wire x1="73.66" y1="25.4" x2="73.66" y2="22.86" width="0.1524" layer="91"/>
+<label x="73.66" y="22.86" size="1.016" layer="95" ratio="10" rot="R180" xref="yes"/>
+</segment>
+</net>
